Commit message: add multiple wheels

File: urdf/track_robot.urdf.xacro (robot description, xacro)
@@ -1,61 +1,31 @@
 <?xml version="1.0"?>
-<robot xmlns:xacro="http://www.ros.org/wiki/xacro" name="track_robot" >
-  <xacro:include filename="$(find track_robot_description)/urdf/common.urdf.xacro" />
-  <xacro:include filename="$(find track_robot_description)/urdf/materials.urdf.xacro" />
-  <xacro:macro name="wheel" params="name parent *origin">
-    <joint name="${name}_joint" type="continuous" >
-      <parent link="${parent}" />
-      <child link="${name}" />
-      <xacro:insert_block name="origin" />
-      <axis xyz="0 0 1" rpy="0 0 0" />
-      <limit effort="30" velocity="0.2" />
-    </joint>
-    <link name="${name}">
-      <visual>
-        <!-- <origin xyz="0 0 -${M_PI/2}" rpy="0 ${M_PI/2} 0" /> -->
-        <geometry>
-          <cylinder radius="0.1" length="0.1" />
-        </geometry>
-        <material name="LightGrey2"/>
-      </visual>
-      <collision >
-        <!-- <origin xyz="0 0 -${M_PI/2}" rpy="0 ${M_PI/2} 0" /> -->
-        <geometry>
-          <cylinder radius="0.11" length="0.11" />
-        </geometry>
-      </collision>
-    </link>
-    <transmission name="${name}_trans" type="SimpleTransmission">
-			<type>transmission_interface/SimpleTransmission</type>
-			<actuator name="${name}_motor">
-				<mechanicalReduction>1</mechanicalReduction>
-			</actuator>
-			<joint name="${name}_joint">
-				<hardwareInterface>hardware_interface/VelocityJointInterface</hardwareInterface>
-			</joint>
-		</transmission>
-  </xacro:macro>
-  <!-- <link name="map" />
-    <origin xyz="0 0 0" rpy="0 0 0" />
-  </link>
-  <joint name="$map_base_joint" type="floating" >
-    <parent link="map" />
-    <child link="base_link" />
-    <origin xyz="0 0 ${0.1/2}" rpy="0 0 0" />
-  </joint> -->
-  <link name="base_link" >
-    <origin xyz="0 0 ${0.1/2 + 0.1}" rpy="0 0 0" />
-    <visual>
-      <geometry>
-        <box size="0.4 0.4 0.1" />
-      </geometry>
-      <material name="Black"/>
-    </visual>
-  </link>
-	<xacro:wheel name="left_wheel" parent="base_link" >
-		<origin xyz="0 0.2 0" rpy="-${M_PI/2} 0 0" />
-	</xacro:wheel>
-  <xacro:wheel name="right_wheel" parent="base_link" >
-		<origin xyz="0 -0.2 0" rpy="-${M_PI/2} 0 0" />
-	</xacro:wheel>
+<robot xmlns:xacro="http://www.ros.org/wiki/xacro" name="track_robot">
+<!--common-->
+<xacro:include filename="$(find track_robot_description)/urdf/common.urdf.xacro" />
+<xacro:include filename="$(find track_robot_description)/urdf/materials.urdf.xacro" />
+<xacro:include filename="$(find track_robot_description)/urdf/track.urdf.xacro" />
+<!--<link name="map" >
+<origin xyz="0 0 0" rpy="0 0 0" />
+</link>
+<joint name="$map_base_joint" type="fixed" >
+<parent link="map" />
+<child link="base_link" />
+<origin xyz="0 0 ${0.1/2}" rpy="0 0 0" />
+</joint>-->
+<xacro:property name="box_length" value="0.4"/>
+<link name="base_link" >
+<origin xyz="0 0 ${0.1/2 + 0.1}" rpy="0 0 0" />
+<visual>
+<geometry>
+<box size="${box_length} ${box_length} 0.1" />
+</geometry>
+<material name="Black"/>
+</visual>
+</link>
+<xacro:track name="left_track" parent="base_link" length="${box_length}" spin="-${M_PI/2}" >
+<origin xyz="0 0.2 0" rpy="0 ${M_PI/2} 0" />
+</xacro:track>
+<xacro:track name="right_track" parent="base_link" length="${box_length}" spin="${M_PI/2}" >
+<origin xyz="0 -0.2 0" rpy="${M_PI} ${M_PI/2} 0" />
+</xacro:track>
 </robot>
